Commit message: Added R2D2 robot simulation and circular motion script

File: install/urdf_tutorial/share/urdf_tutorial/urdf/02-two-link.urdf (robot description, URDF)
Before this commit: robot two_link_robot, 3 links, 2 joints
Links:
- removed link world
- link base_link: geometry visual cylinder length=0.2 radius=0.6
- link link1: geometry visual box size=0.6 0.6 0.1
Joints:
- removed joint world_to_base
- joint base_to_link1: limit lower=-3.14 upper=3.14 effort=1 velocity=1 -> lower=-3.14 upper=3.14 effort=10 velocity=1
